Commit message: NO delay in odom with lidar, joint is publishing but direction is wrong - before break

File: src/nexva_description/urdf/nexva.urdf.xacro (robot description, xacro)
@@ -7,5 +7,8 @@
     <parent link="base_footprint"/>
     <child link="base_link"/>
-    <origin xyz="0 0 0" rpy="0 0 1.507"/>
+    <!-- base_footprint is base_link projected on the ground: same heading,
+         so this joint carries no rotation. Mounting yaw for the lidar belongs
+         in lidar_joint, not here. -->
+    <origin xyz="0 0 0" rpy="0 0 0"/>
   </joint>
 <link name="base_link">

Commit message: urdf tf is working

File: src/nexva_description/urdf/nexva.urdf.xacro (robot description, xacro)
@@ -7,8 +7,10 @@
     <parent link="base_footprint"/>
     <child link="base_link"/>
-    <!-- base_footprint is base_link projected on the ground: same heading,
-         so this joint carries no rotation. Mounting yaw for the lidar belongs
-         in lidar_joint, not here. -->
-    <origin xyz="0 0 0" rpy="0 0 0"/>
+    <!-- The meshes and wheel joints were authored with the robot driving along
+         an axis that is not +X (both wheels sit at x = +-0.12, so the axle
+         runs along X). ROS expects +X forward, so base_link is yawed here to
+         correct it: -90 deg squared the model up, plus a further 180 deg to
+         face it the right way round, giving +90 deg total. -->
+    <origin xyz="0 0 0" rpy="0 0 1.5708"/>
   </joint>
 <link name="base_link">
@@ -21,5 +23,5 @@
     <origin xyz="0 0 0.07" rpy="0 0 0"/>
     <geometry>
-      <mesh filename="file://$(find nexva_description)/meshes/base_link.stl" scale="0.001 0.001 0.001"/>
+      <mesh filename="package://nexva_description/meshes/base_link.stl" scale="0.001 0.001 0.001"/>
     </geometry>
     <material name="green"/>
@@ -28,5 +30,5 @@
     <origin xyz="0 0 0.07" rpy="0 0 0"/>
     <geometry>
-      <mesh filename="file://$(find nexva_description)/meshes/base_link.stl" scale="0.001 0.001 0.001"/>
+      <mesh filename="package://nexva_description/meshes/base_link.stl" scale="0.001 0.001 0.001"/>
     </geometry>
   </collision>
@@ -41,5 +43,5 @@
     <origin xyz="0 0 0" rpy="0 0 0"/>
     <geometry>
-      <mesh filename="file://$(find nexva_description)/meshes/laser.stl" scale="0.001 0.001 0.001"/>
+      <mesh filename="package://nexva_description/meshes/lidar_1.stl" scale="0.001 0.001 0.001"/>
     </geometry>
     <material name="blue"/>
@@ -48,5 +50,5 @@
     <origin xyz="0 0 0" rpy="0 0 0"/>
     <geometry>
-      <mesh filename="file://$(find nexva_description)/meshes/laser.stl" scale="0.001 0.001 0.001"/>
+      <mesh filename="package://nexva_description/meshes/lidar_1.stl" scale="0.001 0.001 0.001"/>
     </geometry>
   </collision>
@@ -61,5 +63,5 @@
     <origin xyz="0 0 0" rpy="0 0 0"/>
     <geometry>
-      <mesh filename="file://$(find nexva_description)/meshes/left_wheel_1.stl" scale="0.001 0.001 0.001"/>
+      <mesh filename="package://nexva_description/meshes/left_wheel_1.stl" scale="0.001 0.001 0.001"/>
     </geometry>
     <material name="black"/>
@@ -68,5 +70,5 @@
     <origin xyz="0 0 0" rpy="0 0 0"/>
     <geometry>
-      <mesh filename="file://$(find nexva_description)/meshes/left_wheel_1.stl" scale="0.001 0.001 0.001"/>
+      <mesh filename="package://nexva_description/meshes/left_wheel_1.stl" scale="0.001 0.001 0.001"/>
     </geometry>
   </collision>
@@ -81,5 +83,5 @@
     <origin xyz="0 0 0" rpy="0 0 0"/>
     <geometry>
-      <mesh filename="file://$(find nexva_description)/meshes/right_wheel_1.stl" scale="0.001 0.001 0.001"/>
+      <mesh filename="package://nexva_description/meshes/right_wheel_1.stl" scale="0.001 0.001 0.001"/>
     </geometry>
     <material name="black"/>
@@ -88,5 +90,5 @@
     <origin xyz="0 0 0" rpy="0 0 0"/>
     <geometry>
-      <mesh filename="file://$(find nexva_description)/meshes/right_wheel_1.stl" scale="0.001 0.001 0.001"/>
+      <mesh filename="package://nexva_description/meshes/right_wheel_1.stl" scale="0.001 0.001 0.001"/>
     </geometry>
   </collision>
@@ -98,5 +100,5 @@
 </joint>
 <joint name="left_wheel_joint" type="continuous">
-  <origin xyz="-0.12 0 0.0317" rpy="0 1.5708 1.5708"/>
+  <origin xyz="0.12 0 0.0317" rpy="0 1.5708 1.5708"/>
   <parent link="base_link"/>
   <child link="left_wheel_1"/>
@@ -104,5 +106,5 @@
 </joint>
 <joint name="right_wheel_joint" type="continuous">
-  <origin xyz="0.12 0 0.0317" rpy="0 1.5708 1.5708"/>
+  <origin xyz="-0.12 0 0.0317" rpy="0 1.5708 1.5708"/>
   <parent link="base_link"/>
   <child link="right_wheel_1"/>

Commit message: robot model

File: src/nexva_description/urdf/nexva.urdf.xacro (robot description, xacro)
@@ -20,6 +20,9 @@
     <inertia ixx="0.040343" iyy="0.056755" izz="0.029008" ixy="1.8e-05" iyz="1e-05" ixz="-0.0"/>
   </inertial>
+  <!-- The STLs were exported Y-up (base_link.stl measures 0.270 x 0.145 x
+       0.270, so its thin axis is Y). ROS is Z-up, so the mesh is rolled +90
+       deg about X here. The wheel joints already do this via their own rpy. -->
   <visual>
-    <origin xyz="0 0 0.07" rpy="0 0 0"/>
+    <origin xyz="0 0 0.07" rpy="1.5708 0 0"/>
     <geometry>
       <mesh filename="package://nexva_description/meshes/base_link.stl" scale="0.001 0.001 0.001"/>
@@ -28,5 +31,5 @@
   </visual>
   <collision>
-    <origin xyz="0 0 0.07" rpy="0 0 0"/>
+    <origin xyz="0 0 0.07" rpy="1.5708 0 0"/>
     <geometry>
       <mesh filename="package://nexva_description/meshes/base_link.stl" scale="0.001 0.001 0.001"/>
@@ -41,5 +44,5 @@
   </inertial>
   <visual>
-    <origin xyz="0 0 0" rpy="0 0 0"/>
+    <origin xyz="0 0 -0.087" rpy="1.5708 0 0"/>
     <geometry>
       <mesh filename="package://nexva_description/meshes/lidar_1.stl" scale="0.001 0.001 0.001"/>
@@ -48,5 +51,5 @@
   </visual>
   <collision>
-    <origin xyz="0 0 0" rpy="0 0 0"/>
+    <origin xyz="0 0 -0.087" rpy="1.5708 0 0"/>
     <geometry>
       <mesh filename="package://nexva_description/meshes/lidar_1.stl" scale="0.001 0.001 0.001"/>
@@ -95,5 +98,9 @@
 </link>
 <joint name="lidar_joint" type="fixed">
-  <origin xyz="0 0 0.07" rpy="0 0 1.5708 "/>
+  <!-- 0.157 puts the scanner flush on the chassis top: the body reaches
+       z=0.1445 and lidar_1.stl carries a baked 0.087 m offset, so this is the
+       height the CAD assembly had it at. The laser frame must sit at the real
+       scanner centre, since that is where the scan originates. -->
+  <origin xyz="0 0 0.157" rpy="0 0 1.5708 "/>
   <parent link="base_link"/>
   <child link="laser"/>
